File: bootstrap.kicad_sch (KiCad schematic)
At the start: 30 parts, among them U130 PCF8574_0x20, U131 PCF8574_0x21, U132 PCF8574_0x22, U133 PCF8574_0x23, U134 PCF8574_0x24, U135 PCF8574_0x25, U136 PCF8574_0x26, U137 PCF8574_0x27, U138 PCF8574A_0x38, U139 PCF8574A_0x39, U140 PCF8574A_0x3A, U141 PCF8574A_0x3B, U142 PCF8574A_0x3C, U143 PCF8574A_0x3D, U144 PCF8574A_0x3E

Commit message: Regenerate KiCad output files for v1.0 architecture
Co-authored-by: Copilot <223556219+Copilot@users.noreply.github.com>
Parts:
- removed C210, C211, C212, C213, C214, C215, C216, C217, C218, C219, C220, C221, C222, C223, C224: 100nF, symbol Device:C
- removed U130: PCF8574_0x20, symbol Interface_I2C:PCF8574
- removed U131: PCF8574_0x21, symbol Interface_I2C:PCF8574
- removed U132: PCF8574_0x22, symbol Interface_I2C:PCF8574
- removed U133: PCF8574_0x23, symbol Interface_I2C:PCF8574
- removed U134: PCF8574_0x24, symbol Interface_I2C:PCF8574
- removed U135: PCF8574_0x25, symbol Interface_I2C:PCF8574
- removed U136: PCF8574_0x26, symbol Interface_I2C:PCF8574
- removed U137: PCF8574_0x27, symbol Interface_I2C:PCF8574
- removed U138: PCF8574A_0x38, symbol Interface_I2C:PCF8574
- removed U139: PCF8574A_0x39, symbol Interface_I2C:PCF8574
- removed U140: PCF8574A_0x3A, symbol Interface_I2C:PCF8574
- removed U141: PCF8574A_0x3B, symbol Interface_I2C:PCF8574
- removed U142: PCF8574A_0x3C, symbol Interface_I2C:PCF8574
- removed U143: PCF8574A_0x3D, symbol Interface_I2C:PCF8574
- removed U144: PCF8574A_0x3E, symbol Interface_I2C:PCF8574
- added C? (x14): 100nF, symbol Device:C
- added U?: PCF8574_0x20, symbol Interface_I2C:PCF8574
- added U?: PCF8574_0x21, symbol Interface_I2C:PCF8574
- added U?: PCF8574_0x22, symbol Interface_I2C:PCF8574
- added U?: PCF8574_0x23, symbol Interface_I2C:PCF8574
- added U?: PCF8574_0x24, symbol Interface_I2C:PCF8574
- added U?: PCF8574_0x25, symbol Interface_I2C:PCF8574
- added U?: PCF8574_0x26, symbol Interface_I2C:PCF8574
- added U?: PCF8574_0x27, symbol Interface_I2C:PCF8574
- added U?: PCF8574A_0x38, symbol Interface_I2C:PCF8574
- added U?: PCF8574A_0x39, symbol Interface_I2C:PCF8574
- added U?: PCF8574A_0x3A, symbol Interface_I2C:PCF8574
- added U?: PCF8574A_0x3B, symbol Interface_I2C:PCF8574
- added U?: PCF8574A_0x3C, symbol Interface_I2C:PCF8574
- added U?: PCF8574A_0x3D, symbol Interface_I2C:PCF8574
Other:
- note added: "14 x 8 = 112 outputs: 110 for worker RESET + 2 spare"
- note added: "8x PCF8574 (0x20-0x27) + 6x PCF8574A (0x38-0x3D) = 14 chips"
- note added: "A0=G A1=G A2=G"
- note added: "A0=G A1=G A2=V"
- note added: "A0=G A1=V A2=G"
- note added: "A0=G A1=V A2=V"
- note added: "A0=V A1=G A2=G"
- note added: "A0=V A1=G A2=V"
- note added: "A0=V A1=V A2=G"
- note added: "A0=V A1=V A2=V"
- note added: "Bootstrap Controller — 14x PCF8574/PCF8574A I2C GPIO Expander"
- note removed: "15 x 8 = 120 outputs, all used for RUN pins"
- note removed: "A0=GND A1=GND A2=GND"
- note removed: "A0=GND A1=GND A2=VCC"
- note removed: "A0=GND A1=VCC A2=GND"
- note removed: "A0=GND A1=VCC A2=VCC"
- note removed: "A0=VCC A1=GND A2=GND"
- note removed: "A0=VCC A1=GND A2=VCC"
- note removed: "A0=VCC A1=VCC A2=GND"
- note removed: "A0=VCC A1=VCC A2=VCC"
- note removed: "Bootstrap Controller — 15x PCF8574/PCF8574A I2C GPIO Expanders"
- note removed: "Pico I2C0 (GP0-1) -> 8x PCF8574 (0x20-0x27) + 7x PCF8574A (0x38-0x3E)"
- note removed: "RUN active-low: pull low = hold in reset, release = boot"
- title: Bootstrap — 15x PCF8574/PCF8574A RUN Pin Control -> Bootstrap — 14x I2C GPIO Expander (CS Mux)
