File: clock_tree.kicad_sch (KiCad schematic)
At the start: 32 parts, among them U145 74HC244, U146 74HC244, U147 74HC244, U148 74HC244, U149 74HC244, U150 74HC244, U151 74HC244, U152 74HC244, U153 74HC244, U154 74HC244, U155 74HC244, U156 74HC244, U157 74HC244, U158 74HC244, U159 74HC244, Y1 12MHz

Commit message: Regenerate KiCad output files for v1.0 architecture
Co-authored-by: Copilot <223556219+Copilot@users.noreply.github.com>
Parts:
- removed C230, C231, C232, C233, C234, C235, C236, C237, C238, C239, C240, C241, C242, C243, C244, C245: 100nF, symbol Device:C
- removed U145, U146, U147, U148, U149, U150, U151, U152, U153, U154, U155, U156, U157, U158, U159: 74HC244, symbol 74xx:74HC244
- removed Y1: 12MHz, symbol Oscillator:ASE
- added C? (x15): 100nF, symbol Device:C
- added U? (x14): 74HC244, symbol 74xx:74HC244
- added Y?: 12MHz, symbol Oscillator:ASE
Other:
- note added: "14 x 8 = 112 buffered outputs, 110 used for workers"
- note added: "1x 12MHz CMOS oscillator -> 14x 74HC244 octal buffers"
- note added: "Clock Fanout Tree — 110 nodes"
- note removed: "15 x 8 = 120 outputs, all used -> each worker XIN pin"
- note removed: "1x 12MHz CMOS oscillator (SiT8008/Abracon ASE, 4-pin, 2.5x2.0mm)"
- note removed: "Clock Fanout Tree"
- note removed: "Output drives 15x 74HC244 octal buffers (8 outputs each)"
- title: Clock Tree — 12MHz Oscillator + 15x 74HC244 Fanout -> Clock Tree — 1x Oscillator + 14x Buffer
