File: cluster_board.kicad_sch (KiCad schematic)
At the start: 13 parts, among them J1 PICO_UART, J10 TILE_OUT_1, J11 TILE_OUT_2, J12 TILE_OUT_3, J13 TILE_OUT_4, J14 TILE_OUT_5, J15 TILE_OUT_6, J2 BOOT_I2C, J3 TILE_IN

Commit message: Regenerate KiCad output files for v1.0 architecture
Co-authored-by: Copilot <223556219+Copilot@users.noreply.github.com>
Parts:
- removed D2: SYS, symbol Device:LED
- removed D3: ERR, symbol Device:LED
- removed J1: PICO_UART, symbol Connector:Pico_UART_Header
- removed J10: TILE_OUT_1, symbol Connector:Grove_SPI
- removed J11: TILE_OUT_2, symbol Connector:Grove_SPI
- removed J12: TILE_OUT_3, symbol Connector:Grove_SPI
- removed J13: TILE_OUT_4, symbol Connector:Grove_SPI
- removed J14: TILE_OUT_5, symbol Connector:Grove_SPI
- removed J15: TILE_OUT_6, symbol Connector:Grove_SPI
- removed J2: BOOT_I2C, symbol Connector:Grove_I2C
- removed J3: TILE_IN, symbol Connector:Grove_SPI
- removed R2, R3: 1k, symbol Device:R
- added D?: PWR_Green, symbol Device:LED
- added D?: SYS_Blue, symbol Device:LED
- added D?: ERR_Red, symbol Device:LED
- added D?: NET_Yellow, symbol Device:LED
- added J?: RJ45_PoE, symbol Connector:RJ45_PoE
- added J?: USB_C, symbol Connector:USB_C_Receptacle
- added J?: GROVE_I2C, symbol Connector:Grove_I2C
- added J?: 12V_DC, symbol Connector:Screw_Terminal_01x02
- added R? (x2): 5.1k, symbol Device:R
- added R? (x4): 330, symbol Device:R
Other:
- sheet Node_13 renamed Worker_13
- sheet Node_16 renamed Worker_18
- sheet Node_19 renamed Worker_23
- sheet Node_22 renamed Worker_28
- sheet Node_62 renamed Worker_95
- sheet Node_65 renamed Worker_100
- sheet Node_68 renamed Worker_105
- removed sheet Node_1
- removed sheet Node_10
- removed sheet Node_100
- removed sheet Node_101
- removed sheet Node_102
- removed sheet Node_103
- removed sheet Node_104
- removed sheet Node_105
- removed sheet Node_106
- removed sheet Node_107
- removed sheet Node_108
- removed sheet Node_109
- removed sheet Node_11
- removed sheet Node_110
- removed sheet Node_111
- removed sheet Node_112
- removed sheet Node_113
- removed sheet Node_114
- removed sheet Node_115
- removed sheet Node_116
- removed sheet Node_117
- removed sheet Node_118
- removed sheet Node_119
- removed sheet Node_12
- removed sheet Node_120
- removed sheet Node_14
- removed sheet Node_15
- removed sheet Node_17
- removed sheet Node_18
- removed sheet Node_2
- removed sheet Node_20
- removed sheet Node_21
- removed sheet Node_23
- removed sheet Node_24
- removed sheet Node_25
- removed sheet Node_26
- removed sheet Node_27
- removed sheet Node_28
- removed sheet Node_29
- removed sheet Node_3
- removed sheet Node_30
- removed sheet Node_31
- removed sheet Node_32
- removed sheet Node_33
- removed sheet Node_34
- removed sheet Node_35
- removed sheet Node_36
- removed sheet Node_37
- removed sheet Node_38
- removed sheet Node_39
- removed sheet Node_4
- removed sheet Node_40
- removed sheet Node_41
- removed sheet Node_42
- removed sheet Node_43
- removed sheet Node_44
- removed sheet Node_45
- removed sheet Node_46
- removed sheet Node_47
- removed sheet Node_48
- removed sheet Node_49
- removed sheet Node_5
- removed sheet Node_50
- removed sheet Node_51
- removed sheet Node_52
- removed sheet Node_53
- removed sheet Node_54
- removed sheet Node_55
- removed sheet Node_56
- removed sheet Node_57
- removed sheet Node_58
- removed sheet Node_59
- removed sheet Node_6
- removed sheet Node_60
- removed sheet Node_61
- removed sheet Node_63
- removed sheet Node_64
- removed sheet Node_66
- removed sheet Node_67
- removed sheet Node_69
- removed sheet Node_7
- removed sheet Node_70
- removed sheet Node_71
- removed sheet Node_72
- removed sheet Node_73
- removed sheet Node_74
- removed sheet Node_75
- removed sheet Node_76
- removed sheet Node_77
- removed sheet Node_78
- removed sheet Node_79
- removed sheet Node_8
- removed sheet Node_80
- removed sheet Node_81
- removed sheet Node_82
- removed sheet Node_83
- removed sheet Node_84
- removed sheet Node_85
- removed sheet Node_86
- removed sheet Node_87
- removed sheet Node_88
- removed sheet Node_89
- removed sheet Node_9
- removed sheet Node_90
- removed sheet Node_91
- removed sheet Node_92
- removed sheet Node_93
- removed sheet Node_94
- removed sheet Node_95
- removed sheet Node_96
- removed sheet Node_97
- removed sheet Node_98
- removed sheet Node_99
- added sheet FPGA_Subsystem (fpga_subsystem.kicad_sch)
- added sheet Worker_0 (worker_node.kicad_sch)
- added sheet Worker_1 (worker_node.kicad_sch)
- added sheet Worker_10 (worker_node.kicad_sch)
- added sheet Worker_101 (worker_node.kicad_sch)
- added sheet Worker_102 (worker_node.kicad_sch)
- added sheet Worker_103 (worker_node.kicad_sch)
- added sheet Worker_104 (worker_node.kicad_sch)
- added sheet Worker_106 (worker_node.kicad_sch)
- added sheet Worker_107 (worker_node.kicad_sch)
- added sheet Worker_108 (worker_node.kicad_sch)
- added sheet Worker_109 (worker_node.kicad_sch)
- added sheet Worker_11 (worker_node.kicad_sch)
- added sheet Worker_12 (worker_node.kicad_sch)
- added sheet Worker_14 (worker_node.kicad_sch)
- added sheet Worker_15 (worker_node.kicad_sch)
- added sheet Worker_16 (worker_node.kicad_sch)
- added sheet Worker_17 (worker_node.kicad_sch)
- added sheet Worker_19 (worker_node.kicad_sch)
- added sheet Worker_2 (worker_node.kicad_sch)
- added sheet Worker_20 (worker_node.kicad_sch)
- added sheet Worker_21 (worker_node.kicad_sch)
- added sheet Worker_22 (worker_node.kicad_sch)
- added sheet Worker_24 (worker_node.kicad_sch)
- added sheet Worker_25 (worker_node.kicad_sch)
- added sheet Worker_26 (worker_node.kicad_sch)
- added sheet Worker_27 (worker_node.kicad_sch)
- added sheet Worker_29 (worker_node.kicad_sch)
- added sheet Worker_3 (worker_node.kicad_sch)
- added sheet Worker_30 (worker_node.kicad_sch)
- added sheet Worker_31 (worker_node.kicad_sch)
- added sheet Worker_32 (worker_node.kicad_sch)
- added sheet Worker_33 (worker_node.kicad_sch)
- added sheet Worker_34 (worker_node.kicad_sch)
- added sheet Worker_35 (worker_node.kicad_sch)
- added sheet Worker_36 (worker_node.kicad_sch)
- added sheet Worker_37 (worker_node.kicad_sch)
- added sheet Worker_38 (worker_node.kicad_sch)
- added sheet Worker_39 (worker_node.kicad_sch)
- added sheet Worker_4 (worker_node.kicad_sch)
- added sheet Worker_40 (worker_node.kicad_sch)
- added sheet Worker_41 (worker_node.kicad_sch)
- added sheet Worker_42 (worker_node.kicad_sch)
- added sheet Worker_43 (worker_node.kicad_sch)
- added sheet Worker_44 (worker_node.kicad_sch)
- added sheet Worker_45 (worker_node.kicad_sch)
- added sheet Worker_46 (worker_node.kicad_sch)
- added sheet Worker_47 (worker_node.kicad_sch)
- added sheet Worker_48 (worker_node.kicad_sch)
- added sheet Worker_49 (worker_node.kicad_sch)
- added sheet Worker_5 (worker_node.kicad_sch)
- added sheet Worker_50 (worker_node.kicad_sch)
- added sheet Worker_51 (worker_node.kicad_sch)
- added sheet Worker_52 (worker_node.kicad_sch)
- added sheet Worker_53 (worker_node.kicad_sch)
- added sheet Worker_54 (worker_node.kicad_sch)
- added sheet Worker_55 (worker_node.kicad_sch)
- added sheet Worker_56 (worker_node.kicad_sch)
- added sheet Worker_57 (worker_node.kicad_sch)
- added sheet Worker_58 (worker_node.kicad_sch)
- added sheet Worker_59 (worker_node.kicad_sch)
- added sheet Worker_6 (worker_node.kicad_sch)
- added sheet Worker_60 (worker_node.kicad_sch)
- added sheet Worker_61 (worker_node.kicad_sch)
- added sheet Worker_62 (worker_node.kicad_sch)
- added sheet Worker_63 (worker_node.kicad_sch)
- added sheet Worker_64 (worker_node.kicad_sch)
- added sheet Worker_65 (worker_node.kicad_sch)
- added sheet Worker_66 (worker_node.kicad_sch)
- added sheet Worker_67 (worker_node.kicad_sch)
- added sheet Worker_68 (worker_node.kicad_sch)
- added sheet Worker_69 (worker_node.kicad_sch)
- added sheet Worker_7 (worker_node.kicad_sch)
- added sheet Worker_70 (worker_node.kicad_sch)
- added sheet Worker_71 (worker_node.kicad_sch)
- added sheet Worker_72 (worker_node.kicad_sch)
- added sheet Worker_73 (worker_node.kicad_sch)
- added sheet Worker_74 (worker_node.kicad_sch)
- added sheet Worker_75 (worker_node.kicad_sch)
- added sheet Worker_76 (worker_node.kicad_sch)
- added sheet Worker_77 (worker_node.kicad_sch)
- added sheet Worker_78 (worker_node.kicad_sch)
- added sheet Worker_79 (worker_node.kicad_sch)
- added sheet Worker_8 (worker_node.kicad_sch)
- added sheet Worker_80 (worker_node.kicad_sch)
- added sheet Worker_81 (worker_node.kicad_sch)
- added sheet Worker_82 (worker_node.kicad_sch)
- added sheet Worker_83 (worker_node.kicad_sch)
- added sheet Worker_84 (worker_node.kicad_sch)
- added sheet Worker_85 (worker_node.kicad_sch)
- added sheet Worker_86 (worker_node.kicad_sch)
- added sheet Worker_87 (worker_node.kicad_sch)
- added sheet Worker_88 (worker_node.kicad_sch)
- added sheet Worker_89 (worker_node.kicad_sch)
- added sheet Worker_9 (worker_node.kicad_sch)
- added sheet Worker_90 (worker_node.kicad_sch)
- added sheet Worker_91 (worker_node.kicad_sch)
- added sheet Worker_92 (worker_node.kicad_sch)
- added sheet Worker_93 (worker_node.kicad_sch)
- added sheet Worker_94 (worker_node.kicad_sch)
- added sheet Worker_96 (worker_node.kicad_sch)
- added sheet Worker_97 (worker_node.kicad_sch)
- added sheet Worker_98 (worker_node.kicad_sch)
- added sheet Worker_99 (worker_node.kicad_sch)
- sheet Bootstrap ports: added I2C_SCL, I2C_SDA; removed BOOT_I2C_SCL, BOOT_I2C_SDA, RUN_N1, RUN_N10, RUN_N100, RUN_N101, RUN_N102, RUN_N103, RUN_N104, RUN_N105, RUN_N106, RUN_N107, RUN_N108, RUN_N109, RUN_N11, RUN_N110, RUN_N111, RUN_N112, RUN_N113, RUN_N114, RUN_N115, RUN_N116, RUN_N117, RUN_N118, RUN_N119, RUN_N12, RUN_N120, RUN_N13, RUN_N14, RUN_N15, RUN_N16, RUN_N17, RUN_N18, RUN_N19, RUN_N2, RUN_N20, RUN_N21, RUN_N22, RUN_N23, RUN_N24, RUN_N25, RUN_N26, RUN_N27, RUN_N28, RUN_N29, RUN_N3, RUN_N30, RUN_N31, RUN_N32, RUN_N33, RUN_N34, RUN_N35, RUN_N36, RUN_N37, RUN_N38, RUN_N39, RUN_N4, RUN_N40, RUN_N41, RUN_N42, RUN_N43, RUN_N44, RUN_N45, RUN_N46, RUN_N47, RUN_N48, RUN_N49, RUN_N5, RUN_N50, RUN_N51, RUN_N52, RUN_N53, RUN_N54, RUN_N55, RUN_N56, RUN_N57, RUN_N58, RUN_N59, RUN_N6, RUN_N60, RUN_N61, RUN_N62, RUN_N63, RUN_N64, RUN_N65, RUN_N66, RUN_N67, RUN_N68, RUN_N69, RUN_N7, RUN_N70, RUN_N71, RUN_N72, RUN_N73, RUN_N74, RUN_N75, RUN_N76, RUN_N77, RUN_N78, RUN_N79, RUN_N8, RUN_N80, RUN_N81, RUN_N82, RUN_N83, RUN_N84, RUN_N85, RUN_N86, RUN_N87, RUN_N88, RUN_N89, RUN_N9, RUN_N90, RUN_N91, RUN_N92, RUN_N93, RUN_N94, RUN_N95, RUN_N96, RUN_N97, RUN_N98, RUN_N99
- sheet Clock_Tree ports: added none; removed CLK_12M_N1, CLK_12M_N10, CLK_12M_N100, CLK_12M_N101, CLK_12M_N102, CLK_12M_N103, CLK_12M_N104, CLK_12M_N105, CLK_12M_N106, CLK_12M_N107, CLK_12M_N108, CLK_12M_N109, CLK_12M_N11, CLK_12M_N110, CLK_12M_N111, CLK_12M_N112, CLK_12M_N113, CLK_12M_N114, CLK_12M_N115, CLK_12M_N116, CLK_12M_N117, CLK_12M_N118, CLK_12M_N119, CLK_12M_N12, CLK_12M_N120, CLK_12M_N13, CLK_12M_N14, CLK_12M_N15, CLK_12M_N16, CLK_12M_N17, CLK_12M_N18, CLK_12M_N19, CLK_12M_N2, CLK_12M_N20, CLK_12M_N21, CLK_12M_N22, CLK_12M_N23, CLK_12M_N24, CLK_12M_N25, CLK_12M_N26, CLK_12M_N27, CLK_12M_N28, CLK_12M_N29, CLK_12M_N3, CLK_12M_N30, CLK_12M_N31, CLK_12M_N32, CLK_12M_N33, CLK_12M_N34, CLK_12M_N35, CLK_12M_N36, CLK_12M_N37, CLK_12M_N38, CLK_12M_N39, CLK_12M_N4, CLK_12M_N40, CLK_12M_N41, CLK_12M_N42, CLK_12M_N43, CLK_12M_N44, CLK_12M_N45, CLK_12M_N46, CLK_12M_N47, CLK_12M_N48, CLK_12M_N49, CLK_12M_N5, CLK_12M_N50, CLK_12M_N51, CLK_12M_N52, CLK_12M_N53, CLK_12M_N54, CLK_12M_N55, CLK_12M_N56, CLK_12M_N57, CLK_12M_N58, CLK_12M_N59, CLK_12M_N6, CLK_12M_N60, CLK_12M_N61, CLK_12M_N62, CLK_12M_N63, CLK_12M_N64, CLK_12M_N65, CLK_12M_N66, CLK_12M_N67, CLK_12M_N68, CLK_12M_N69, CLK_12M_N7, CLK_12M_N70, CLK_12M_N71, CLK_12M_N72, CLK_12M_N73, CLK_12M_N74, CLK_12M_N75, CLK_12M_N76, CLK_12M_N77, CLK_12M_N78, CLK_12M_N79, CLK_12M_N8, CLK_12M_N80, CLK_12M_N81, CLK_12M_N82, CLK_12M_N83, CLK_12M_N84, CLK_12M_N85, CLK_12M_N86, CLK_12M_N87, CLK_12M_N88, CLK_12M_N89, CLK_12M_N9, CLK_12M_N90, CLK_12M_N91, CLK_12M_N92, CLK_12M_N93, CLK_12M_N94, CLK_12M_N95, CLK_12M_N96, CLK_12M_N97, CLK_12M_N98, CLK_12M_N99, CLK_12M_SRC
- sheet Power_Supply ports: added POE_VIN_N, POE_VIN_P, VCC_3V3_Z1, VCC_3V3_Z2, VCC_3V3_Z3, VCC_3V3_Z4, VIN_12V; removed VCC_12V, VCC_3V3_A, VCC_3V3_B
- sheet Worker_100 ports: added CLK_IN, RESET, SPI_CS, SPI_MISO, SPI_MOSI, SPI_SCK; removed CLK_12M, RUN, SPI_DN_CS, SPI_DN_MISO, SPI_DN_MOSI, SPI_DN_SCK, SPI_UP_CS, SPI_UP_MISO, SPI_UP_MOSI, SPI_UP_SCK, SWCLK, SWDIO, UART_RX, UART_TX
- sheet Worker_105 ports: added CLK_IN, RESET, SPI_CS, SPI_MISO, SPI_MOSI, SPI_SCK; removed CLK_12M, RUN, SPI_DN_CS, SPI_DN_MISO, SPI_DN_MOSI, SPI_DN_SCK, SPI_UP_CS, SPI_UP_MISO, SPI_UP_MOSI, SPI_UP_SCK, SWCLK, SWDIO, UART_RX, UART_TX
- sheet Worker_13 ports: added CLK_IN, RESET, SPI_CS, SPI_MISO, SPI_MOSI, SPI_SCK; removed CLK_12M, RUN, SPI_DN_CS, SPI_DN_MISO, SPI_DN_MOSI, SPI_DN_SCK, SPI_UP_CS, SPI_UP_MISO, SPI_UP_MOSI, SPI_UP_SCK, SWCLK, SWDIO, UART_RX, UART_TX
- sheet Worker_18 ports: added CLK_IN, RESET, SPI_CS, SPI_MISO, SPI_MOSI, SPI_SCK; removed CLK_12M, RUN, SPI_DN_CS, SPI_DN_MISO, SPI_DN_MOSI, SPI_DN_SCK, SPI_UP_CS, SPI_UP_MISO, SPI_UP_MOSI, SPI_UP_SCK, SWCLK, SWDIO, UART_RX, UART_TX
- sheet Worker_23 ports: added CLK_IN, RESET, SPI_CS, SPI_MISO, SPI_MOSI, SPI_SCK; removed CLK_12M, RUN, SPI_DN_CS, SPI_DN_MISO, SPI_DN_MOSI, SPI_DN_SCK, SPI_UP_CS, SPI_UP_MISO, SPI_UP_MOSI, SPI_UP_SCK, SWCLK, SWDIO, UART_RX, UART_TX
- sheet Worker_28 ports: added CLK_IN, RESET, SPI_CS, SPI_MISO, SPI_MOSI, SPI_SCK; removed CLK_12M, RUN, SPI_DN_CS, SPI_DN_MISO, SPI_DN_MOSI, SPI_DN_SCK, SPI_UP_CS, SPI_UP_MISO, SPI_UP_MOSI, SPI_UP_SCK, SWCLK, SWDIO, UART_RX, UART_TX
- sheet Worker_95 ports: added CLK_IN, RESET, SPI_CS, SPI_MISO, SPI_MOSI, SPI_SCK; removed CLK_12M, RUN, SPI_DN_CS, SPI_DN_MISO, SPI_DN_MOSI, SPI_DN_SCK, SPI_UP_CS, SPI_UP_MISO, SPI_UP_MOSI, SPI_UP_SCK, SWCLK, SWDIO, UART_RX, UART_TX
- note added: "110x RP2354B (220 cores) | iCE40HX4K FPGA SPI star | W5500 Ethernet"
- note added: "12V DC input (or PoE)"
- note added: "14x PCF8574/PCF8574A (112 bootstrap outputs, 110 used)"
- note added: "1x Oscillator + 14x 74HC244 (112 clocks, 110 used)"
- note added: "4x TPS54560 + PoE PD (Ag9905)"
- note added: "4x TPS54560 | 14x PCF8574 | 14x 74HC244 | 14x 74HC595 | PoE 802.3af"
- note added: "5.1k on CC1/CC2 to GND (UFP sink)"
- note added: "5x MicroSD RAID-0 | 200x200mm 4-layer PCB"
- note added: "CS_0..CS_109: individual chip selects from FPGA 74HC595 cascade"
- note added: "ETH signals: FPGA subsystem <-> RJ45 MagJack"
- note added: "Global buses: VCC_3V3, I2C (SDA/SCL), SPI (MOSI/MISO/SCK)"
- note added: "I2C bootstrap bus connector"
- note added: "PWR | SYS | ERR | NET LEDs (330 ohm)"
- note added: "PoE center taps: RJ45 CT1/CT2 -> Power Supply Ag9905"
- note added: "RJ45 MagJack with PoE center taps"
- note added: "RP2354 110-Node Network Compute Fabric v1.0"
- note added: "W0"
- note added: "W1"
- note added: "W10"
- note added: "W100"
- note added: "W101"
- note added: "W102"
- note added: "W103"
- note added: "W104"
- note added: "W105"
- note added: "W106"
- note added: "W107"
- note added: "W108"
- note added: "W109"
- note added: "W11"
- note added: "W12"
- note added: "W13"
- note added: "W14"
- note added: "W15"
- note added: "W16"
- note added: "W17"
- note added: "W18"
- note added: "W19"
- note added: "W2"
- note added: "W20"
- note added: "W21"
- note added: "W22"
- note added: "W23"
- note added: "W24"
- note added: "W25"
- note added: "W26"
- note added: "W27"
- note added: "W28"
- note added: "W29"
- note added: "W3"
- note added: "W30"
- note added: "W31"
- note added: "W32"
- note added: "W33"
- note added: "W34"
- note added: "W35"
- note added: "W36"
- note added: "W37"
- note added: "W38"
- note added: "W39"
- note added: "W4"
- note added: "W40"
- note added: "W41"
- note added: "W42"
- note added: "W43"
- note added: "W44"
- note added: "W45"
- note added: "W46"
- note added: "W47"
- note added: "W48"
- note added: "W49"
- note added: "W5"
- note added: "W50"
- note added: "W51"
- note added: "W52"
- note added: "W53"
- note added: "W54"
- note added: "W55"
- note added: "W56"
- note added: "W57"
- note added: "W58"
- note added: "W59"
- note added: "W6"
- note added: "W60"
- note added: "W61"
- note added: "W62"
- note added: "W63"
- note added: "W64"
- note added: "W65"
- note added: "W66"
- note added: "W67"
- note added: "W68"
- note added: "W69"
- note added: "W7"
- note added: "W70"
- note added: "W71"
- note added: "W72"
- note added: "W73"
- note added: "W74"
- note added: "W75"
- note added: "W76"
- note added: "W77"
- note added: "W78"
- note added: "W79"
- note added: "W8"
- note added: "W80"
- note added: "W81"
- note added: "W82"
- note added: "W83"
- note added: "W84"
- note added: "W85"
- note added: "W86"
- note added: "W87"
- note added: "W88"
- note added: "W89"
- note added: "W9"
- note added: "W90"
- note added: "W91"
- note added: "W92"
- note added: "W93"
- note added: "W94"
- note added: "W95"
- note added: "W96"
- note added: "W97"
- note added: "W98"
- note added: "W99"
- note added: "iCE40HX4K + W5500 + 5x MicroSD + 2x Cache + 14x 74HC595"
- note removed: "10 UART chains x 12 nodes | Dual TPS54560 from 12V | 4-layer 200x200mm PCB"
- note removed: "120x RP2354B (ALL QFN-80) | SPI data pipeline between nodes"
- note removed: "12MHz Oscillator + 15x 74HC244 (120 clocks)"
- note removed: "15x PCF8574/A bootstrap | 15x 74HC244 clock | SPI Grove inter-tile"
- note removed: "15x PCF8574/PCF8574A Bootstrap (120 RUN outputs)"
- note removed: "6x TILE_OUT -> 6-way tree topology"
- note removed: "Chain A: Pico GP2->TX-> N1..N12 ->RX->GP3 Pico"
- note removed: "Chain B: Pico GP4->TX-> N13..N24 ->RX->GP5 Pico"
- note removed: "Chain C: Pico GP6->TX-> N25..N36 ->RX->GP7 Pico"
- note removed: "Chain D: Pico GP8->TX-> N37..N48 ->RX->GP9 Pico"
- note removed: "Chain E: Pico GP10->TX-> N49..N60 ->RX->GP11 Pico"
- note removed: "Chain F: Pico GP12->TX-> N61..N72 ->RX->GP13 Pico"
- note removed: "Chain G: Pico GP14->TX-> N73..N84 ->RX->GP15 Pico"
- note removed: "Chain H: Pico GP16->TX-> N85..N96 ->RX->GP17 Pico"
- note removed: "Chain I: Pico GP18->TX-> N97..N108 ->RX->GP19 Pico"
- note removed: "Chain J: Pico GP20->TX-> N109..N120 ->RX->GP21 Pico"
- note removed: "Jumper wires to breadboard Pico 2 (26/26 GPIO used)"
- note removed: "N1 (RP2354B)"
- note removed: "N10 (RP2354B)"
- note removed: "N100 (RP2354B)"
- note removed: "N101 (RP2354B)"
- note removed: "N102 (RP2354B)"
- note removed: "N103 (RP2354B)"
- note removed: "N104 (RP2354B)"
- note removed: "N105 (RP2354B)"
- note removed: "N106 (RP2354B)"
- note removed: "N107 (RP2354B)"
- note removed: "N108 (RP2354B)"
- note removed: "N109 (RP2354B)"
- note removed: "N11 (RP2354B)"
- note removed: "N110 (RP2354B)"
- note removed: "N111 (RP2354B)"
- note removed: "N112 (RP2354B)"
- note removed: "N113 (RP2354B)"
- note removed: "N114 (RP2354B)"
- note removed: "N115 (RP2354B)"
- note removed: "N116 (RP2354B)"
- note removed: "N117 (RP2354B)"
- note removed: "N118 (RP2354B)"
- note removed: "N119 (RP2354B)"
- note removed: "N12 (RP2354B)"
- note removed: "N120 (RP2354B)"
- note removed: "N13 (RP2354B)"
- note removed: "N14 (RP2354B)"
- note removed: "N15 (RP2354B)"
- note removed: "N16 (RP2354B)"
- note removed: "N17 (RP2354B)"
- note removed: "N18 (RP2354B)"
- note removed: "N19 (RP2354B)"
- note removed: "N2 (RP2354B)"
- note removed: "N20 (RP2354B)"
- note removed: "N21 (RP2354B)"
- note removed: "N22 (RP2354B)"
- note removed: "N23 (RP2354B)"
- note removed: "N24 (RP2354B)"
- note removed: "N25 (RP2354B)"
- note removed: "N26 (RP2354B)"
- note removed: "N27 (RP2354B)"
- note removed: "N28 (RP2354B)"
- note removed: "N29 (RP2354B)"
- note removed: "N3 (RP2354B)"
- note removed: "N30 (RP2354B)"
- note removed: "N31 (RP2354B)"
- note removed: "N32 (RP2354B)"
- note removed: "N33 (RP2354B)"
- note removed: "N34 (RP2354B)"
- note removed: "N35 (RP2354B)"
- note removed: "N36 (RP2354B)"
- note removed: "N37 (RP2354B)"
- note removed: "N38 (RP2354B)"
- note removed: "N39 (RP2354B)"
- note removed: "N4 (RP2354B)"
- note removed: "N40 (RP2354B)"
- note removed: "N41 (RP2354B)"
- note removed: "N42 (RP2354B)"
- note removed: "N43 (RP2354B)"
- note removed: "N44 (RP2354B)"
- note removed: "N45 (RP2354B)"
- note removed: "N46 (RP2354B)"
- note removed: "N47 (RP2354B)"
- note removed: "N48 (RP2354B)"
- note removed: "N49 (RP2354B)"
- note removed: "N5 (RP2354B)"
- note removed: "N50 (RP2354B)"
- note removed: "N51 (RP2354B)"
- note removed: "N52 (RP2354B)"
- note removed: "N53 (RP2354B)"
- note removed: "N54 (RP2354B)"
- note removed: "N55 (RP2354B)"
- note removed: "N56 (RP2354B)"
- note removed: "N57 (RP2354B)"
- note removed: "N58 (RP2354B)"
- note removed: "N59 (RP2354B)"
- note removed: "N6 (RP2354B)"
- note removed: "N60 (RP2354B)"
- note removed: "N61 (RP2354B)"
- note removed: "N62 (RP2354B)"
- note removed: "N63 (RP2354B)"
- note removed: "N64 (RP2354B)"
- note removed: "N65 (RP2354B)"
- note removed: "N66 (RP2354B)"
- note removed: "N67 (RP2354B)"
- note removed: "N68 (RP2354B)"
- note removed: "N69 (RP2354B)"
- note removed: "N7 (RP2354B)"
- note removed: "N70 (RP2354B)"
- note removed: "N71 (RP2354B)"
- note removed: "N72 (RP2354B)"
- note removed: "N73 (RP2354B)"
- note removed: "N74 (RP2354B)"
- note removed: "N75 (RP2354B)"
- note removed: "N76 (RP2354B)"
- note removed: "N77 (RP2354B)"
- note removed: "N78 (RP2354B)"
- note removed: "N79 (RP2354B)"
- note removed: "N8 (RP2354B)"
- note removed: "N80 (RP2354B)"
- note removed: "N81 (RP2354B)"
- note removed: "N82 (RP2354B)"
- note removed: "N83 (RP2354B)"
- note removed: "N84 (RP2354B)"
- note removed: "N85 (RP2354B)"
- note removed: "N86 (RP2354B)"
- note removed: "N87 (RP2354B)"
- note removed: "N88 (RP2354B)"
- note removed: "N89 (RP2354B)"
- note removed: "N9 (RP2354B)"
- note removed: "N90 (RP2354B)"
- note removed: "N91 (RP2354B)"
- note removed: "N92 (RP2354B)"
- note removed: "N93 (RP2354B)"
- note removed: "N94 (RP2354B)"
- note removed: "N95 (RP2354B)"
- note removed: "N96 (RP2354B)"
- note removed: "N97 (RP2354B)"
- note removed: "N98 (RP2354B)"
- note removed: "N99 (RP2354B)"
- note removed: "Pico I2C0 (GP0/GP1)"
- note removed: "RP2354 Cluster Tile v0.6"
- note removed: "SYS LED on Pico GP22 (active low) | ERR LED on Pico GP26 (active low)"
- note removed: "Shared worker I2C control bus: all 120 workers + Pico GP27-28 (I2C1)"
- note removed: "Upstream SPI from parent tile"
- title: RP2354 120-Node Compute Tile v0.6  -> RP2354 110-Node Network Compute Fabric v1.0
